File: KiCAD/circuit/adapter.kicad_pcb (KiCad board)
At the start: 2 copper layers, 13 parts, among them J1 Pin header, J2 Pin header, U1 PIC16f1825-I/P, U2 MCP2515-I/P, U3 MCP2561-E/P, Y1 Ceralock 8MHz

Commit message: update
Parts:
- added D1: 1A, diode:diode, F.Cu at (212.1, 101.6)
- added F1: 250mA, polyswitch:polyswitch, F.Cu at (152.4, 88.9)
- added J3: Pin header, Connector_PinHeader_2.54mm:PinHeader_1x4_L_Shape, F.Cu at (142.2, 96.5)
- moved R1 61.5 mm to (195.6, 137.2)
- moved C2 54.9 mm to (113.0, 67.3)
- moved JP1 51.2 mm to (119.4, 100.3)
- moved C3 49.3 mm to (165.1, 58.4)
- moved R2 38.8 mm to (123.2, 87.6), turned to 180 degrees
- moved R3 32.1 mm to (171.4, 82.5)
- moved Y1 30.0 mm to (110.5, 61.0)
- moved U1 29.5 mm to (127.0, 81.3)
- moved U3 26.2 mm to (151.1, 67.3)
- moved J1 25.0 mm to (120.7, 92.7)
- moved U2 24.0 mm to (129.5, 67.3)
- moved C1 20.7 mm to (165.1, 130.8)
- moved J2 13.3 mm to (158.8, 105.4)
Connections:
- J1 pad 1: +5V -> Net-(F1-Pad2)
- J1 pad 2: GND -> Net-(D1-Pad1)
- J2 pad 1: Net-(J2-Pad1) -> +5V
- J2 pad 2: Net-(J2-Pad2) -> GND
- J2 pad 3: Net-(J2-Pad1) -> Net-(J2-Pad3)
- J2 pad 4: Net-(J2-Pad2) -> Net-(J2-Pad4)
- JP1 pad 1: Net-(J2-Pad2) -> Net-(J2-Pad4)
- R1 pad 1: Net-(J2-Pad1) -> Net-(J2-Pad3)
- U3 pad 6: Net-(J2-Pad2) -> Net-(J2-Pad4)
- U3 pad 7: Net-(J2-Pad1) -> Net-(J2-Pad3)
Other:
- rule pad_to_mask_clearance: 0.2 -> 0

Commit message: update
Parts:
- added C4: 47u, can-bus:Capacitor_2.54mm, F.Cu at (116.2, 123.8)
- added C5: 0.1u, can-bus:Capacitor_2.54mm, F.Cu at (104.8, 129.5)
- added D2: 1A, can-bus:Diode, F.Cu at (132.1, 108.6)
- added D3: LED, can-bus:Led, F.Cu at (118.1, 80.6)
- added F2: 250mA, can-bus:Polyswitch_Tyco, F.Cu at (111.1, 137.2)
- added J4: CAN0, can-bus:PinHeader_1x2_L_Shape, F.Cu at (207.6, 125.7)
- added J5: CAN1, can-bus:PinHeader_1x2_L_Shape, F.Cu at (200.0, 126.4)
- added J6: ICSP, can-bus:PinSocket_1x6, F.Cu at (141.0, 90.2)
- added J7: terminal, can-bus:Terminal_PhoenixContact_2P, F.Cu at (125.1, 137.8)
- added JP2: Jumper, can-bus:Jumper_1x2, F.Cu at (116.2, 88.3)
- added R5: 1k, can-bus:Resistor_FaithfulLink_CF25, F.Cu at (114.9, 74.3)
- added SW1: SW, can-bus:TactileSwitch, F.Cu at (125.1, 89.5)
- added U4: regulator, can-bus:TA48M05F, F.Cu at (118.7, 129.5)
- C1, C2, C3: footprint Murata_Capacitor:Capacitor -> can-bus:Capacitor_2.54mm
- D1: footprint diode:diode -> can-bus:Diode
- F1: footprint polyswitch:polyswitch -> can-bus:Polyswitch_Tyco
- J1: footprint Connector_PinHeader_2.54mm:PinHeader_1x4_L_Shape -> can-bus:PinHeader_1x4_L_Shape
- J2, J3: value Pin header -> Pin socket; footprint Connector_PinHeader_2.54mm:PinHeader_1x4_L_Shape -> can-bus:PinSocket_1x4
- JP1: footprint Connector_PinHeader_2.54mm:Jumper_1x2 -> can-bus:Jumper_1x2
- R1, R2, R3: footprint Resistor:Resistor_FaithfulLink_CF25 -> can-bus:Resistor_FaithfulLink_CF25
- U1: value PIC16f1825-I/P -> PIC16f18326-I/P; footprint IC_Sockets:IC_socket_14pins -> can-bus:IC_socket_14pins
- U2: value MCP2515-I/P -> MCP2561-E/P; footprint IC_Sockets:IC_socket_18pins -> can-bus:IC_Socket_8pins
- U3: value MCP2561-E/P -> MCP2515-I/P; footprint IC_Sockets:IC_Socket_8pins -> can-bus:IC_socket_18pins
- Y1: footprint Murata_Ceralock:Ceralock -> can-bus:Ceralock_Murata
- moved D1 99.5 mm to (113.7, 116.2)
- moved JP1 92.2 mm to (210.8, 111.8)
- moved Y1 88.0 mm to (181.0, 113.7)
- moved U2 83.5 mm to (200.7, 111.1)
- moved U3 64.6 mm to (183.5, 123.2)
- moved C3 61.9 mm to (191.8, 114.3)
- moved R3 50.6 mm to (188.6, 130.2)
- moved C2 37.6 mm to (148.0, 81.3)
- moved C1 36.7 mm to (200.0, 119.4)
- moved J2 30.3 mm to (130.2, 95.2)
- moved J1 29.8 mm to (143.5, 111.8)
- moved R1 24.7 mm to (212.1, 118.7)
- moved J3 24.3 mm to (134.0, 73.7)
- moved R2 24.0 mm to (143.5, 74.9), turned to 0 degrees
- moved U1 8.98 mm to (135.9, 82.5), turned to 0 degrees
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Connections:
- D1 pad 1: Net-(D1-Pad1) -> +5V
- J1 pad 2: Net-(D1-Pad1) -> GND
- J2 pad 1: +5V -> Net-(J2-Pad1)
- J2 pad 2: GND -> Net-(J2-Pad2)
- J2 pad 3: Net-(J2-Pad3) -> GND
- J2 pad 4: Net-(J2-Pad4) -> +5V
- J3 pad 1: +5V -> Net-(J3-Pad1)
- J3 pad 2: GND -> Net-(J3-Pad2)
- J3 pad 3: Net-(J2-Pad3) -> Net-(J3-Pad3)
- J3 pad 4: Net-(J2-Pad4) -> Net-(J3-Pad4)
- JP1 pad 1: Net-(J2-Pad4) -> Net-(J4-Pad2)
- R1 pad 1: Net-(J2-Pad3) -> Net-(J4-Pad1)
- R2 pad 2: Net-(R2-Pad2) -> Net-(J3-Pad4)
- U1 pad 2: Net-(U1-Pad2) -> Net-(J2-Pad2)
- U1 pad 3: Net-(U1-Pad3) -> Net-(J2-Pad1)
- U1 pad 4: Net-(R2-Pad2) -> Net-(J3-Pad4)
- U1 pad 5: Net-(U1-Pad5) -> Net-(J3-Pad3)
- U1 pad 6: Net-(U1-Pad6) -> Net-(J3-Pad2)
- U1 pad 7: Net-(U1-Pad7) -> Net-(J3-Pad1)
- U2 pad 2: Net-(U2-Pad2) -> GND
- U2 pad 3: Net-(U2-Pad3) -> +5V
- U2 pad 6: Net-(U2-Pad6) -> Net-(J4-Pad2)
- U2 pad 7: Net-(U2-Pad7) -> Net-(J4-Pad1)
- U2 pad 8: Net-(U2-Pad8) -> GND
- U3 pad 2: GND -> Net-(U2-Pad4)
- U3 pad 3: +5V -> Net-(U3-Pad3)
- U3 pad 4: Net-(U2-Pad2) -> Net-(U3-Pad4)
- U3 pad 6: Net-(J2-Pad4) -> Net-(U3-Pad6)
- U3 pad 7: Net-(J2-Pad3) -> Net-(U3-Pad7)
- U3 pad 8: GND -> Net-(U3-Pad8)
- Y1 pad 1: Net-(U2-Pad8) -> Net-(U3-Pad8)
- Y1 pad 3: Net-(U2-Pad7) -> Net-(U3-Pad7)
Other:
- board outline added: 47.6 x 36.8 mm
