File: KiCAD/circuit/adapter.kicad_pcb (KiCad board)
At the start: 2 copper layers, 47.6 x 36.8 mm, 31 parts, among them J1 Pin header, J2 Pin socket, J3 Pin socket, J4 CAN0, J5 CAN1, J6 ICSP, J7 terminal, SW1 SW, U1 PIC16f18326-I/P, U2 MCP2561-E/P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

Commit message: update
Parts:
- moved U1 0.52 mm to (158.1, 109.2)
- moved C4 0.28 mm to (160.7, 118.1)
- moved R2 0.18 mm to (154.3, 116.2)
Routing:
- net +5V: track 105.9 -> 107.4 mm
- net Net-(J3-Pad4): track 67.4 -> 68.1 mm
- net Net-(J3-Pad3): track 32.8 -> 32.2 mm, vias 0 -> 2
- net Net-(J1-Pad4): track 66.3 -> 65.7 mm
- net Net-(U1-Pad9): track 6.17 -> 5.61 mm
- net Net-(U1-Pad10): track 6.55 -> 6.04 mm
- net Net-(J3-Pad2): track 32.3 -> 32.7 mm, vias 1 -> 0
- added copper zone on F.Cu, net Net-(J2-Pad1)
Other:
- board text added: "SA"

Commit message: update
Parts:
- removed D2: 1A, can-bus:Diode
Routing:
- net Net-(C5-Pad1): track 23.9 -> 15.9 mm
Other:
- board text added: "CAN node v0.2 Apr 15, 2018"
- board text removed: "SA"
Changed lines of the file:
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@@
 (kicad_pcb (version 4) (host pcbnew 4.0.7)
   (general
-    (links 68)
+    (links 66)
     (no_connects 0)
     (area 125.679999 91.389999 173.405001 128.320001)
     (thickness 1.6)
     (drawings 5)
-    (tracks 237)
+    (tracks 234)
     (zones 0)
-    (modules 31)
+    (modules 30)
     (nets 37)
   )
@@
       (outputformat 1)
       (mirror false)
-      (drillshape 1)
+      (drillshape 0)
       (scaleselection 1)
       (outputdirectory ""))
@@
       (net 16 "Net-(J4-Pad2)"))
   )
-  (module can-bus:Diode (layer F.Cu)
-    (at 167.64 116.205)
-    (fp_text reference D2 (at 3.175 -2.54) (layer F.SilkS)
-      (effects (font (size 1 1) (thickness 0.15)))
-    )
-    (fp_text value 1A (at 0 0) (layer F.Fab)
-      (effects (font (size 1 1) (thickness 0.15)))
-    )
-    (fp_line (start -5.08 -1.27) (end -5.08 1.27) (layer F.SilkS) (width 0.15))
-    (fp_line (start -5.08 1.27) (end 5.08 1.27) (layer F.SilkS) (width 0.15))
-    (fp_line (start 5.08 1.27) (end 5.08 -1.27) (layer F.SilkS) (width 0.15))
-    (fp_line (start 5.08 -1.27) (end -5.08 -1.27) (layer F.SilkS) (width 0.15))
-    (pad 1 thru_hole circle (at 3.81 0) (size 1.8 1.8) (drill 1) (layers *.Cu *.Mask)
-      (net 3 "Net-(C5-Pad1)"))
-    (pad 2 thru_hole circle (at -3.81 0) (size 1.8 1.8) (drill 1) (layers *.Cu *.Mask)
-      (net 1 GND))
-  )
   (module can-bus:Resistor_FaithfulLink_CF25 (layer F.Cu)
     (at 133.985 108.585 90)
@@
       (net 1 GND))
   )
-  (gr_text SA (at 127.635 104.775) (layer B.Cu)
-    (effects (font (size 1.5 1.5) (thickness 0.3)))
+  (gr_text "CAN node v0.2\nApr 15, 2018" (at 167.64 116.205) (layer F.SilkS)
+    (effects (font (size 0.9 0.9) (thickness 0.2)))
   )
   (gr_line (start 173.355 91.44) (end 125.73 91.44) (angle 90) (layer Edge.Cuts) (width 0.1))
@@
   (gr_line (start 125.73 128.27) (end 173.355 128.27) (angle 90) (layer Edge.Cuts) (width 0.1))
   (gr_line (start 125.73 91.44) (end 125.73 128.27) (angle 90) (layer Edge.Cuts) (width 0.1))
-  (segment (start 150.495 113.03) (end 150.495 116.205) (width 0.25) (layer F.Cu) (net 2) (status C00000))
-  (segment (start 150.495 116.205) (end 152.4 118.11) (width 0.25) (layer F.Cu) (net 2) (status 400000))
+  (segment (start 150.495 113.03) (end 150.495 116.205) (width 0.25) (layer F.Cu) (net 2))
+  (segment (start 150.495 116.205) (end 152.4 118.11) (width 0.25) (layer F.Cu) (net 2))
   (segment (start 152.4 118.11) (end 159.385 118.11) (width 0.25) (layer F.Cu) (net 2))
-  (segment (start 159.385 118.11) (end 160.655 119.38) (width 0.25) (layer F.Cu) (net 2) (status 800000))
-  (segment (start 160.655 119.38) (end 160.655 123.19) (width 0.25) (layer F.Cu) (net 2) (status C00000))
-  (segment (start 160.655 119.38) (end 162.56 117.475) (width 0.25) (layer F.Cu) (net 2) (status 400000))
+  (segment (start 159.385 118.11) (end 160.655 119.38) (width 0.25) (layer F.Cu) (net 2))
+  (segment (start 160.655 119.38) (end 160.655 123.19) (width 0.25) (layer F.Cu) (net 2))
+  (segment (start 160.655 119.38) (end 162.56 117.475) (width 0.25) (layer F.Cu) (net 2))
   (segment (start 162.56 117.475) (end 162.56 115.57) (width 0.25) (layer F.Cu) (net 2))
   (segment (start 162.56 115.57) (end 163.83 114.3) (width 0.25) (layer F.Cu) (net 2))
@@
   (segment (start 166.37 114.3) (end 167.005 113.665) (width 0.25) (layer F.Cu) (net 2))
   (segment (start 167.005 113.665) (end 167.005 108.585) (width 0.25) (layer F.Cu) (net 2))
-  (segment (start 167.005 108.585) (end 171.45 104.14) (width 0.25) (layer F.Cu) (net 2) (status 800000))
+  (segment (start 167.005 108.585) (end 171.45 104.14) (width 0.25) (layer F.Cu) (net 2))
   (segment (start 150.495 113.03) (end 150.495 113.665) (width 0.25) (layer F.Cu) (net 2))
   (segment (start 150.495 113.665) (end 148.59 115.57) (width 0.25) (layer F.Cu) (net 2))
@@
   (segment (start 135.89 121.92) (end 135.89 119.38) (width 0.25) (layer F.Cu) (net 2))
   (segment (start 158.115 126.365) (end 160.02 124.46) (width 0.25) (layer F.Cu) (net 3))
-  (segment (start 165.1 120.65) (end 165.1 118.745) (width 0.25) (layer F.Cu) (net 3))
+  (segment (start 165.1 120.65) (end 165.1 118.745) (width 0.25) (layer F.Cu) (net 3) (status 20))
   (segment (start 161.29 124.46) (end 165.1 120.65) (width 0.25) (layer F.Cu) (net 3))
   (segment (start 160.02 124.46) (end 161.29 124.46) (width 0.25) (layer F.Cu) (net 3))
@@
   (segment (start 155.575 124.46) (end 157.48 126.365) (width 0.25) (layer F.Cu) (net 3))
   (segment (start 157.48 126.365) (end 158.115 126.365) (width 0.25) (layer F.Cu) (net 3))
-  (segment (start 165.1 118.745) (end 167.64 116.205) (width 0.25) (layer F.Cu) (net 3))
-  (segment (start 167.64 116.205) (end 171.45 116.205) (width 0.25) (layer F.Cu) (net 3))
-  (segment (start 170.815 116.205) (end 171.45 116.205) (width 0.25) (layer F.Cu) (net 3) (status 30))
   (segment (start 139.7 104.14) (end 143.51 104.14) (width 0.25) (layer F.Cu) (net 4))
   (segment (start 143.51 104.14) (end 144.78 102.87) (width 0.25) (layer F.Cu) (net 4))
@@
   (segment (start 130.81 121.92) (end 132.08 121.92) (width 0.25) (layer F.Cu) (net 6))
   (segment (start 132.08 121.92) (end 134.62 124.46) (width 0.25) (layer F.Cu) (net 6))
-  (segment (start 170.18 118.745) (end 170.18 124.46) (width 0.25) (layer F.Cu) (net 7))
+  (segment (start 170.18 118.745) (end 170.18 124.46) (width 0.25) (layer F.Cu) (net 7) (status 10))
   (segment (start 151.765 95.885) (end 153.035 97.155) (width 0.25) (layer B.Cu) (net 8))
   (via (at 151.765 95.885) (size 0.6) (drill 0.4) (layers F.Cu B.Cu) (net 8))
@@
   (segment (start 130.175 118.11) (end 141.605 118.11) (width 0.25) (layer B.Cu) (net 12))
   (segment (start 128.27 116.205) (end 130.175 118.11) (width 0.25) (layer B.Cu) (net 12))
-  (segment (start 152.4 116.205) (end 158.115 116.205) (width 0.25) (layer B.Cu) (net 12) (status 800000))
+  (segment (start 152.4 116.205) (end 158.115 116.205) (width 0.25) (layer B.Cu) (net 12))
   (segment (start 150.495 118.11) (end 152.4 116.205) (width 0.25) (layer B.Cu) (net 12))
-  (segment (start 158.115 113.03) (end 158.115 116.205) (width 0.25) (layer F.Cu) (net 12) (status C00000))
+  (segment (start 158.115 113.03) (end 158.115 116.205) (width 0.25) (layer F.Cu) (net 12))
   (segment (start 157.988 116.078) (end 158.115 116.205) (width 0.25) (layer F.Cu) (net 12) (status 30))
   (segment (start 151.13 109.22) (end 154.305 109.22) (width 0.25) (layer F.Cu) (net 12))

Commit message: update
Parts:
- moved J2 1.91 mm to (132.1, 98.4)
- moved R5 1.42 mm to (134.6, 107.3)
- renumbered SW1 to Reset
Routing:
- net +5V: track 107.4 -> 105.8 mm
- net Net-(U2-Pad4): track 46.4 -> 45.1 mm
- net Net-(J2-Pad1): track 25.7 -> 26.9 mm
- net Net-(J2-Pad2): track 30.2 -> 29.1 mm, vias 3 -> 1
- net Net-(J3-Pad1): track 36.3 -> 37.3 mm
- net Net-(U2-Pad1): track 41.3 -> 40.4 mm
- removed copper zone on F.Cu, net Net-(J2-Pad1)
Other:
- board text added: "+"
- board text added: "5V"
- board text added: "6-18V"
- board text added: "Expansion board"
- board text added: "GND"
- board text added: "H"
- board text added: "ICSP"
- board text added: "L"
- board text added: "MCP2515"
- board text added: "MCP2561"
- board text added: "PIC MCU"
- board text added: "RX"
- board text added: "TX"

Commit message: update
Routing:
- net Net-(J3-Pad4): track 68.1 -> 69.9 mm
Changed lines of the file:
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@@
     (thickness 1.6)
     (drawings 27)
-    (tracks 214)
+    (tracks 213)
     (zones 0)
     (modules 30)
@@
   (module can-bus:Ceralock_Murata (layer F.Cu)
     (at 146.05 92.71)
-    (fp_text reference Y1 (at 0.635 2.54) (layer F.SilkS)
+    (fp_text reference Y1 (at 1.27 1.905) (layer F.SilkS)
       (effects (font (size 1 1) (thickness 0.15)))
     )
@@
       (net 11 "Net-(J2-Pad1)"))
   )
-  (module can-bus:TactileSwitch (layer F.Cu)
-    (at 144.78 98.425)
-    (fp_text reference Reset (at -3.81 -1.905) (layer F.SilkS)
-      (effects (font (size 1 1) (thickness 0.15)))
-    )
-    (fp_text value SW (at 0 2.54) (layer F.Fab)
-      (effects (font (size 1 1) (thickness 0.15)))
-    )
-    (fp_line (start 3.81 -1.27) (end -3.81 -1.27) (layer F.SilkS) (width 0.15))
-    (fp_line (start -3.81 -1.27) (end -3.81 1.27) (layer F.SilkS) (width 0.15))
-    (fp_line (start -3.81 1.27) (end 3.81 1.27) (layer F.SilkS) (width 0.15))
-    (fp_line (start 3.81 1.27) (end 3.81 -1.27) (layer F.SilkS) (width 0.15))
-    (pad 2 thru_hole circle (at -2.54 0) (size 1.8 1.8) (drill 1) (layers *.Cu *.Mask)
-      (net 1 GND))
-    (pad 1 thru_hole circle (at 2.54 0) (size 1.8 1.8) (drill 1) (layers *.Cu *.Mask)
-      (net 12 "Net-(J3-Pad4)"))
-  )
   (module can-bus:Led (layer F.Cu)
     (at 146.05 102.87)
-    (fp_text reference D3 (at 1.27 -1.905) (layer F.SilkS)
+    (fp_text reference D3 (at 1.27 2.54) (layer F.SilkS)
       (effects (font (size 1 1) (thickness 0.15)))
     )
@@
   (module can-bus:Jumper_1x2 (layer F.Cu)
     (at 138.43 101.6 270)
-    (fp_text reference JP2 (at -2.54 -0.635 360) (layer F.SilkS)
+    (fp_text reference JP2 (at -0.635 -3.81 360) (layer F.SilkS)
       (effects (font (size 1 1) (thickness 0.15)))
     )
@@
     (pad 2 thru_hole circle (at -3.81 0) (size 1.8 1.8) (drill 1) (layers *.Cu *.Mask)
       (net 1 GND))
+  )
+  (module can-bus:TactileSwitch (layer F.Cu)
+    (at 144.78 98.425)
+    (fp_text reference Reset (at 0 -2.54) (layer F.SilkS)
+      (effects (font (size 1 1) (thickness 0.15)))
+    )
+    (fp_text value SW (at 0 2.54) (layer F.Fab)
+      (effects (font (size 1 1) (thickness 0.15)))
+    )
+    (fp_line (start -5.08 1.27) (end 5.08 1.27) (layer F.SilkS) (width 0.15))
+    (fp_line (start -5.08 -1.27) (end 5.08 -1.27) (layer F.SilkS) (width 0.15))
+    (fp_line (start -5.08 -1.27) (end -5.08 1.27) (layer F.SilkS) (width 0.15))
+    (fp_line (start 5.08 1.27) (end 5.08 -1.27) (layer F.SilkS) (width 0.15))
+    (pad 2 thru_hole circle (at -3.81 0) (size 1.8 1.8) (drill 1) (layers *.Cu *.Mask)
+      (net 1 GND))
+    (pad 1 thru_hole circle (at 3.81 0) (size 1.8 1.8) (drill 1) (layers *.Cu *.Mask)
+      (net 12 "Net-(J3-Pad4)"))
   )
   (gr_text GND (at 165.1 127) (layer F.SilkS)
@@
   (segment (start 151.765 95.885) (end 153.035 97.155) (width 0.25) (layer B.Cu) (net 8))
   (via (at 151.765 95.885) (size 0.6) (drill 0.4) (layers F.Cu B.Cu) (net 8))
-  (segment (start 143.51 95.885) (end 151.765 95.885) (width 0.25) (layer F.Cu) (net 8))
-  (via (at 143.51 95.885) (size 0.6) (drill 0.4) (layers F.Cu B.Cu) (net 8))
-  (segment (start 135.255 95.885) (end 143.51 95.885) (width 0.25) (layer B.Cu) (net 8))
+  (segment (start 141.605 95.885) (end 151.765 95.885) (width 0.25) (layer F.Cu) (net 8))
+  (via (at 141.605 95.885) (size 0.6) (drill 0.4) (layers F.Cu B.Cu) (net 8))
+  (segment (start 135.255 95.885) (end 141.605 95.885) (width 0.25) (layer B.Cu) (net 8))
   (segment (start 132.715 93.345) (end 135.255 95.885) (width 0.25) (layer B.Cu) (net 8) (status 10))
   (segment (start 153.035 97.155) (end 153.035 105.41) (width 0.25) (layer B.Cu) (net 8))
@@
   (segment (start 154.305 96.52) (end 155.575 97.79) (width 0.25) (layer B.Cu) (net 9))
   (segment (start 155.575 97.79) (end 155.575 105.41) (width 0.25) (layer B.Cu) (net 9))
-  (segment (start 144.78 96.52) (end 154.305 96.52) (width 0.25) (layer F.Cu) (net 9))
+  (segment (start 142.24 96.52) (end 154.305 96.52) (width 0.25) (layer F.Cu) (net 9))
   (via (at 154.305 96.52) (size 0.6) (drill 0.4) (layers F.Cu B.Cu) (net 9))
   (segment (start 129.54 124.46) (end 129.54 121.285) (width 0.25) (layer F.Cu) (net 9))
@@
   (segment (start 129.54 124.46) (end 129.54 123.825) (width 0.25) (layer F.Cu) (net 9) (status 30))
   (segment (start 130.175 93.345) (end 133.35 96.52) (width 0.25) (layer B.Cu) (net 9) (status 10))
-  (via (at 144.78 96.52) (size 0.6) (drill 0.4) (layers F.Cu B.Cu) (net 9))
-  (segment (start 133.35 96.52) (end 144.78 96.52) (width 0.25) (layer B.Cu) (net 9))
+  (via (at 142.24 96.52) (size 0.6) (drill 0.4) (layers F.Cu B.Cu) (net 9))
+  (segment (start 133.35 96.52) (end 142.24 96.52) (width 0.25) (layer B.Cu) (net 9))
   (segment (start 154.305 96.52) (end 154.305 96.52) (width 0.25) (layer B.Cu) (net 9))
   (segment (start 155.702 105.283) (end 155.575 105.41) (width 0.25) (layer B.Cu) (net 9) (status 30))
@@
   (segment (start 138.43 102.87) (end 141.605 102.87) (width 0.25) (layer B.Cu) (net 11))
   (segment (start 135.89 100.33) (end 138.43 102.87) (width 0.25) (layer B.Cu) (net 11))
+  (segment (start 140.335 93.345) (end 140.335 95.885) (width 0.25) (layer F.Cu) (net 12) (status 400000))
+  (segment (start 142.875 98.425) (end 148.59 98.425) (width 0.25) (layer F.Cu) (net 12) (status 800000))
+  (segment (start 140.335 95.885) (end 142.875 98.425) (width 0.25) (layer F.Cu) (net 12))
+  (segment (start 148.59 98.425) (end 146.05 100.965) (width 0.25) (layer B.Cu) (net 12) (status 400000))
+  (via (at 151.13 109.22) (size 0.6) (drill 0.4) (layers F.Cu B.Cu) (net 12))
+  (segment (start 146.05 104.14) (end 151.13 109.22) (width 0.25) (layer B.Cu) (net 12))
+  (segment (start 146.05 100.965) (end 146.05 104.14) (width 0.25) (layer B.Cu) (net 12))
   (segment (start 148.59 118.11) (end 150.495 118.11) (width 0.25) (layer B.Cu) (net 12))
   (via (at 148.59 118.11) (size 0.6) (drill 0.4) (layers F.Cu B.Cu) (net 12))
@@
   (segment (start 154.305 109.22) (end 158.115 113.03) (width 0.25) (layer F.Cu) (net 12))
   (segment (start 157.988 116.078) (end 158.115 116.205) (width 0.25) (layer B.Cu) (net 12) (status 30))
-  (segment (start 140.335 93.345) (end 140.335 95.885) (width 0.25) (layer F.Cu) (net 12) (status 10))
-  (segment (start 146.05 97.155) (end 147.32 98.425) (width 0.25) (layer F.Cu) (net 12))
-  (segment (start 141.605 97.155) (end 146.05 97.155) (width 0.25) (layer F.Cu) (net 12))
-  (segment (start 140.335 95.885) (end 141.605 97.155) (width 0.25) (layer F.Cu) (net 12))
   (segment (start 157.861 115.951) (end 158.115 116.205) (width 0.25) (layer F.Cu) (net 12) (status 30))
   (segment (start 158.115 116.205) (end 157.861 116.205) (width 0.25) (layer B.Cu) (net 12) (status 30))
-  (segment (start 146.05 99.695) (end 147.32 98.425) (width 0.25) (layer B.Cu) (net 12))
-  (segment (start 146.05 104.14) (end 146.05 99.695) (width 0.25) (layer B.Cu) (net 12))
-  (segment (start 151.13 109.22) (end 146.05 104.14) (width 0.25) (layer B.Cu) (net 12))
-  (via (at 151.13 109.22) (size 0.6) (drill 0.4) (layers F.Cu B.Cu) (net 12))
   (segment (start 151.13 109.22) (end 151.13 109.22) (width 0.25) (layer F.Cu) (net 12))
   (segment (start 160.655 113.03) (end 159.385 111.76) (width 0.25) (layer B.Cu) (net 13))
