File: KiCAD/circuit/adapter.sch (KiCad schematic (older format))
At the start: 5 parts, among them J1 Conn_01x04, J2 Conn_01x04, U1 PIC16f1825-I/P, U2 MCP2515-I/P, U3 MCP2561-E/P

Commit message: circuit
Parts:
- added C1, C2, C3: 0.1u, symbol C_Small
- added JP1: Jumper, symbol Jumper_NO_Small
- added R1: 120, symbol R
- added R2: 51k, symbol R
- added R3: 10k, symbol R
- added Y1: Ceralock 8MHz, symbol Resonator_Small
- J1, J2: value Conn_01x04 -> Pin header
Connections:
- net labels added: 5V, CANH, CANL, RX, TX
- net labels removed: VDD
- wire segments 36 -> 97
- no-connect marks 0 -> 12
Other:
- moved on the sheet: J1, J2, U2, U3

Commit message: KiCAD data update
Connections:
- net labels added: +5V
- wire segments 97 -> 81
- no-connect marks 12 -> 13
Other:
- moved on the sheet: C1, C2, C3, J1, J2, JP1, R1, R2, R3, U3, Y1

Commit message: update
Parts:
- C1, C2, C3: footprint (none) -> Murata_Capacitor:Capacitor
- J1, J2: footprint (none) -> Connector_PinHeader_2.54mm:PinHeader_1x4_L_Shape
- JP1: footprint (none) -> Connector_PinHeader_2.54mm:Jumper_1x2
- R1, R2, R3: footprint (none) -> Resistor:Resistor_FaithfulLink_CF25
- U1: footprint (none) -> IC_Sockets:IC_socket_14pins; symbol PIC16f1825-I/P -> PIC16f1825-I/P-RESCUE-adapter
- U2: footprint (none) -> IC_Sockets:IC_socket_18pins; symbol MCP2515-I/P -> MCP2515-I/P-RESCUE-adapter
- U3: footprint (none) -> IC_Sockets:IC_Socket_8pins; symbol MCP2561-E/P -> MCP2561-E/P-RESCUE-adapter
- Y1: footprint (none) -> Murata_Ceralock:Ceralock
Changed lines of the file:
@@
 $EndDescr
 $Comp
-L MCP2561-E/P U3
+L MCP2561-E/P-RESCUE-adapter U3
 U 1 1 5AC360E7
 P 3150 2450
 F 0 "U3" H 2750 3100 60  0000 C CNN
 F 1 "MCP2561-E/P" H 3000 3000 60  0000 C CNN
-F 2 "" H 3150 2450 60  0001 C CNN
+F 2 "IC_Sockets:IC_Socket_8pins" H 3150 2450 60  0001 C CNN
 F 3 "" H 3150 2450 60  0001 C CNN
 	1    3150 2450
@@
 F 0 "J1" H 9550 5300 50  0000 C CNN
 F 1 "Pin header" H 9550 4800 50  0000 C CNN
-F 2 "" H 9550 5100 50  0001 C CNN
+F 2 "Connector_PinHeader_2.54mm:PinHeader_1x4_L_Shape" H 9550 5100 50  0001 C CNN
 F 3 "" H 9550 5100 50  0001 C CNN
 	1    9550 5100
@@
 F 0 "J2" H 4600 5300 50  0000 C CNN
 F 1 "Pin header" H 4600 4800 50  0000 C CNN
-F 2 "" H 4600 5100 50  0001 C CNN
+F 2 "Connector_PinHeader_2.54mm:PinHeader_1x4_L_Shape" H 4600 5100 50  0001 C CNN
 F 3 "" H 4600 5100 50  0001 C CNN
 	1    4600 5100
@@
 F 0 "R2" V 4580 3550 50  0000 C CNN
 F 1 "51k" V 4500 3550 50  0000 C CNN
-F 2 "" V 4430 3550 50  0001 C CNN
+F 2 "Resistor:Resistor_FaithfulLink_CF25" V 4430 3550 50  0001 C CNN
 F 3 "" H 4500 3550 50  0001 C CNN
 	1    4500 3550
@@
 F 0 "R1" V 4030 5450 50  0000 C CNN
 F 1 "120" V 3950 5450 50  0000 C CNN
-F 2 "" V 3880 5450 50  0001 C CNN
+F 2 "Resistor:Resistor_FaithfulLink_CF25" V 3880 5450 50  0001 C CNN
 F 3 "" H 3950 5450 50  0001 C CNN
 	1    3950 5450
@@
 F 0 "JP1" H 3700 5680 50  0000 C CNN
 F 1 "Jumper" H 3710 5540 50  0000 C CNN
-F 2 "" H 3700 5600 50  0001 C CNN
+F 2 "Connector_PinHeader_2.54mm:Jumper_1x2" H 3700 5600 50  0001 C CNN
 F 3 "" H 3700 5600 50  0001 C CNN
 	1    3700 5600
@@
 F 0 "Y1" H 4775 1925 50  0000 L CNN
 F 1 "Ceralock 8MHz" H 4775 1850 50  0000 L CNN
-F 2 "" H 4625 1850 50  0001 C CNN
+F 2 "Murata_Ceralock:Ceralock" H 4625 1850 50  0001 C CNN
 F 3 "" H 4625 1850 50  0001 C CNN
 	1    4650 1850
@@
 F 0 "R3" V 7480 1350 50  0000 C CNN
 F 1 "10k" V 7400 1350 50  0000 C CNN
-F 2 "" V 7330 1350 50  0001 C CNN
+F 2 "Resistor:Resistor_FaithfulLink_CF25" V 7330 1350 50  0001 C CNN
 F 3 "" H 7400 1350 50  0001 C CNN
 	1    7400 1350
@@
 F 0 "C3" H 5860 2370 50  0000 L CNN
 F 1 "0.1u" H 5860 2220 50  0000 L CNN
-F 2 "" H 5850 2300 50  0001 C CNN
+F 2 "Murata_Capacitor:Capacitor" H 5850 2300 50  0001 C CNN
 F 3 "" H 5850 2300 50  0001 C CNN
 	1    5850 2300
@@
 F 0 "C2" H 5810 3320 50  0000 L CNN
 F 1 "0.1u" H 5810 3170 50  0000 L CNN
-F 2 "" H 5800 3250 50  0001 C CNN
+F 2 "Murata_Capacitor:Capacitor" H 5800 3250 50  0001 C CNN
 F 3 "" H 5800 3250 50  0001 C CNN
 	1    5800 3250
@@
 F 0 "C1" H 1810 2320 50  0000 L CNN
 F 1 "0.1u" H 1810 2170 50  0000 L CNN
-F 2 "" H 1800 2250 50  0001 C CNN
+F 2 "Murata_Capacitor:Capacitor" H 1800 2250 50  0001 C CNN
 F 3 "" H 1800 2250 50  0001 C CNN
 	1    1800 2250
@@
 Connection ~ 4800 3550
 $Comp
-L PIC16f1825-I/P U1
+L PIC16f1825-I/P-RESCUE-adapter U1
 U 1 1 5AC4ED87
 P 5450 4000
 F 0 "U1" H 5050 4550 60  0000 C CNN
 F 1 "PIC16f1825-I/P" H 5350 4450 60  0000 C CNN
-F 2 "" H 5350 4450 60  0001 C CNN
+F 2 "IC_Sockets:IC_socket_14pins" H 5350 4450 60  0001 C CNN
 F 3 "" H 5350 4450 60  0001 C CNN
 	1    5450 4000
@@
 $EndComp
 $Comp
-L MCP2515-I/P U2
+L MCP2515-I/P-RESCUE-adapter U2
 U 1 1 5AC4EED7
 P 5800 1650
 F 0 "U2" H 5400 2300 60  0000 C CNN
 F 1 "MCP2515-I/P" H 5650 2200 60  0000 C CNN
-F 2 "" H 7050 1150 60  0001 C CNN
+F 2 "IC_Sockets:IC_socket_18pins" H 7050 1150 60  0001 C CNN
 F 3 "" H 7050 1150 60  0001 C CNN
 	1    5800 1650

Commit message: update
Parts:
- removed J2: Pin header, Connector_PinHeader_2.54mm:PinHeader_1x4_L_Shape, symbol Conn_01x04
- removed U1: PIC16f1825-I/P, IC_Sockets:IC_socket_14pins, symbol PIC16f1825-I/P-RESCUE-adapter
- added D1: 1A, diode:diode, symbol D
- added F1: 250mA, polyswitch:polyswitch, symbol Polyfuse
- added J2, J3: Pin socket, symbol Conn_01x04_Female
- added J4: CAN0, symbol Conn_01x02
- added J5: CAN1, symbol Conn_01x02
- added J6: ICSP, symbol Conn_01x06_Female
- added U1: PIC16f18326-I/P, IC_Sockets:IC_socket_14pins, symbol PIC16f18326-I/P
Connections:
- net +5V: now also D1.1 (K), F1.1, J2.4 (Pin_4), J6.2 (Pin_2), U1.1 (VDD); no longer J1.1 (Pin_1)
- net GND: now also D1.2 (A), J2.3 (Pin_3), J6.3 (Pin_3), U1.14 (VSS); no longer J1.2 (Pin_2)
- net at JP1.1, U3.6 (CANL): now also J4.2 (Pin_2), J5.2 (Pin_2)
- net at R1.1, U3.7 (CANH): now also J4.1 (Pin_1), J5.1 (Pin_1)
- net at J1.3 (Pin_3): now also J6.5 (Pin_5), U1.12 (RX/AN1/RA1)
- net at J1.4 (Pin_4): now also J6.4 (Pin_4), U1.13 (TX/AN0/RA0)
- net at R2.2: now also J3.4 (Pin_4), J6.1 (Pin_1), U1.4 (RA3/MCLR)
- net at U2.13 (SCK): now also U1.10 (SCK/SCL/AN4/RC0)
- net at U2.16 (~CS~): now also U1.11 (AN2/RA2)
- net at U2.14 (SI): now also U1.8 (SDO/AN6/RC2)
- net at U2.15 (SO): now also U1.9 (SDI/SDA/AN5/RC1)
- new net: F1.2, J1.1 (Pin_1)
- new net: J2.1 (Pin_1), U1.3 (RA4/AN3/SDO)
- new net: J2.2 (Pin_2), U1.2 (RA5)
- new net: J3.1 (Pin_1), U1.7 (RC3/AN7)
- new net: J3.2 (Pin_2), U1.6 (RC4/TX)
- new net: J3.3 (Pin_3), U1.5 (RC5/RX)
- no-connect marks 13 -> 9
Other:
- moved on the sheet: C2, R1, R2

Commit message: update
Parts:
- added C4: 100u, symbol CP
- added C5: 0.1u, symbol C_Small
- added D2: 1A, diode:diode, symbol D
- added D3: LED, symbol LED
- added F2: 250mA, polyswitch:polyswitch, symbol Polyfuse
- added J7: terminal, symbol Screw_Terminal_01x02
- added JP2: Jumper, Connector_PinHeader_2.54mm:Jumper_1x2, symbol Jumper_NO_Small
- added R5: 1k, Resistor:Resistor_FaithfulLink_CF25, symbol R
- added SW1: SW, symbol SW_Push
- added U4: regulator, symbol regulator
Connections:
- net +5V: now also C4.1, JP2.2, U4.2 (OUT)
- net GND: now also J1.2 (Pin_2), C4.2, C5.2, D2.2 (A), J7.2 (Pin_2), SW1.2, U4.3 (GND)
- net at J3.4 (Pin_4), J6.1 (Pin_1), R2.2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: now also SW1.1
- net at J3.1 (Pin_1), U1.7 (RC3/AN7): now also R5.2
- new net: C5.1, D2.1 (K), F2.2, U4.1 (In)
- new net: F2.1, J7.1 (Pin_1)
- new net: D3.1 (K), R5.1
- new net: D3.2 (A), JP2.1
Other:
- moved on the sheet: C1, C2, C3, D1, F1, J1, J2, J3, J4, J5, J6, JP1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

Commit message: update
Parts:
- removed U2: MCP2515-I/P, IC_Sockets:IC_socket_18pins, symbol MCP2515-I/P-RESCUE-adapter
- removed U3: MCP2561-E/P, IC_Sockets:IC_Socket_8pins, symbol MCP2561-E/P-RESCUE-adapter
- added U2: MCP2561-E/P, can-bus:IC_Socket_8pins, symbol MCP2561-E/P
- added U3: MCP2515-I/P, can-bus:IC_socket_18pins, symbol MCP2515-I/P
- C1, C2, C3: footprint Murata_Capacitor:Capacitor -> can-bus:Capacitor_2.54mm
- C4: value 100u -> 47u; footprint (none) -> can-bus:Capacitor_2.54mm
- C5: footprint (none) -> can-bus:Capacitor_2.54mm
- D1, D2: footprint diode:diode -> can-bus:Diode
- D3: footprint (none) -> can-bus:Led
- F1, F2: footprint polyswitch:polyswitch -> can-bus:Polyswitch_Tyco
- J1: footprint Connector_PinHeader_2.54mm:PinHeader_1x4_L_Shape -> can-bus:PinHeader_1x4_L_Shape
- J2, J3: footprint (none) -> can-bus:PinSocket_1x4
- J4, J5: footprint (none) -> can-bus:PinHeader_1x2_L_Shape
- J6: footprint (none) -> can-bus:PinSocket_1x6
- J7: footprint (none) -> can-bus:Terminal_PhoenixContact_2P
- JP1, JP2: footprint Connector_PinHeader_2.54mm:Jumper_1x2 -> can-bus:Jumper_1x2
- R1, R2, R3, R5: footprint Resistor:Resistor_FaithfulLink_CF25 -> can-bus:Resistor_FaithfulLink_CF25
- SW1: footprint (none) -> can-bus:TactileSwitch
- U1: footprint IC_Sockets:IC_socket_14pins -> can-bus:IC_socket_14pins
- U4: footprint (none) -> can-bus:TA48M05F
- Y1: footprint Murata_Ceralock:Ceralock -> can-bus:Ceralock_Murata
Connections:
- net +5V: now also U2.3 (VDD), U3.18 (VDD)
- net GND: now also U2.2 (VSS), U2.8 (STBY), U3.9 (VSS)
- net at J4.2 (Pin_2), J5.2 (Pin_2), JP1.1: now also U2.6 (CANL)
- net at J4.1 (Pin_1), J5.1 (Pin_1), R1.1: now also U2.7 (CANH)
- net at Y1.1: now also U3.8 (OSC1)
- net at Y1.3: now also U3.7 (OSC2)
- net at R3.2: now also U3.17 (RESET)
- net at U1.10 (SCK/SCL/AN4/RC0): now also U3.13 (SCK)
- net at U1.8 (SDO/AN6/RC2): now also U3.14 (SI)
- net at U1.9 (SDI/SDA/AN5/RC1): now also U3.15 (SO)
- net at U1.11 (AN2/RA2): now also U3.16 (CS)
- new net: U2.1 (TXD), U3.1 (TXCAN)
- new net: U2.4 (RXD), U3.2 (RXCAN)
Changed lines of the file:
@@
 EESchema Schematic File Version 2
-LIBS:adapter-rescue
 LIBS:can-bus
 LIBS:power
@@
 encoding utf-8
 Sheet 1 1
-Title "CAN adapter to UART"
-Date "2018-04-04"
-Rev "0.1"
-Comp ""
-Comment1 ""
-Comment2 ""
+Title "CAN node base board"
+Date "2018-04-13"
+Rev "0.2"
+Comp "https://github.com/araobp"
+Comment1 "CAN node base board"
+Comment2 "CAN adapter to UART"
 Comment3 ""
 Comment4 ""
 $EndDescr
-$Comp
-L MCP2561-E/P-RESCUE-adapter U3
-U 1 1 5AC360E7
-P 2400 2550
-F 0 "U3" H 2000 3200 60  0000 C CNN
-F 1 "MCP2561-E/P" H 2250 3100 60  0000 C CNN
-F 2 "IC_Sockets:IC_Socket_8pins" H 2400 2550 60  0001 C CNN
-F 3 "" H 2400 2550 60  0001 C CNN
-	1    2400 2550
-	1    0    0    -1
-$EndComp
 $Comp
 L Conn_01x04 J1
@@
 F 0 "J1" H 8600 5400 50  0000 C CNN
 F 1 "Pin header" H 8600 4900 50  0000 C CNN
-F 2 "Connector_PinHeader_2.54mm:PinHeader_1x4_L_Shape" H 8600 5200 50  0001 C CNN
+F 2 "can-bus:PinHeader_1x4_L_Shape" H 8600 5200 50  0001 C CNN
 F 3 "" H 8600 5200 50  0001 C CNN
 	1    8600 5200
@@
 F 0 "R2" V 3830 3850 50  0000 C CNN
 F 1 "51k" V 3750 3850 50  0000 C CNN
-F 2 "Resistor:Resistor_FaithfulLink_CF25" V 3680 3850 50  0001 C CNN
+F 2 "can-bus:Resistor_FaithfulLink_CF25" V 3680 3850 50  0001 C CNN
 F 3 "" H 3750 3850 50  0001 C CNN
 	1    3750 3850
@@
 F 0 "R1" V 3280 6350 50  0000 C CNN
 F 1 "120" V 3200 6350 50  0000 C CNN
-F 2 "Resistor:Resistor_FaithfulLink_CF25" V 3130 6350 50  0001 C CNN
+F 2 "can-bus:Resistor_FaithfulLink_CF25" V 3130 6350 50  0001 C CNN
 F 3 "" H 3200 6350 50  0001 C CNN
 	1    3200 6350
@@
 F 0 "JP1" H 2950 6680 50  0000 C CNN
 F 1 "Jumper" H 2960 6540 50  0000 C CNN
-F 2 "Connector_PinHeader_2.54mm:Jumper_1x2" H 2950 6600 50  0001 C CNN
+F 2 "can-bus:Jumper_1x2" H 2950 6600 50  0001 C CNN
 F 3 "" H 2950 6600 50  0001 C CNN
 	1    2950 6600
@@
 F 0 "Y1" H 4025 2025 50  0000 L CNN
 F 1 "Ceralock 8MHz" H 4025 1950 50  0000 L CNN
-F 2 "Murata_Ceralock:Ceralock" H 3875 1950 50  0001 C CNN
+F 2 "can-bus:Ceralock_Murata" H 3875 1950 50  0001 C CNN
 F 3 "" H 3875 1950 50  0001 C CNN
 	1    3900 1950
@@
 F 0 "R3" V 6730 1450 50  0000 C CNN
 F 1 "10k" V 6650 1450 50  0000 C CNN
-F 2 "Resistor:Resistor_FaithfulLink_CF25" V 6580 1450 50  0001 C CNN
+F 2 "can-bus:Resistor_FaithfulLink_CF25" V 6580 1450 50  0001 C CNN
 F 3 "" H 6650 1450 50  0001 C CNN
 	1    6650 1450
@@
 F 0 "C3" H 5110 2470 50  0000 L CNN
 F 1 "0.1u" H 5110 2320 50  0000 L CNN
-F 2 "Murata_Capacitor:Capacitor" H 5100 2400 50  0001 C CNN
+F 2 "can-bus:Capacitor_2.54mm" H 5100 2400 50  0001 C CNN
 F 3 "" H 5100 2400 50  0001 C CNN
 	1    5100 2400
@@
 F 0 "C2" H 5060 3620 50  0000 L CNN
 F 1 "0.1u" H 5060 3470 50  0000 L CNN
-F 2 "Murata_Capacitor:Capacitor" H 5050 3550 50  0001 C CNN
+F 2 "can-bus:Capacitor_2.54mm" H 5050 3550 50  0001 C CNN
 F 3 "" H 5050 3550 50  0001 C CNN
 	1    5050 3550
@@
 F 0 "C1" H 1060 2420 50  0000 L CNN
 F 1 "0.1u" H 1060 2270 50  0000 L CNN
-F 2 "Murata_Capacitor:Capacitor" H 1050 2350 50  0001 C CNN
+F 2 "can-bus:Capacitor_2.54mm" H 1050 2350 50  0001 C CNN
 F 3 "" H 1050 2350 50  0001 C CNN
 	1    1050 2350
@@
 $EndComp
 $Comp
-L MCP2515-I/P-RESCUE-adapter U2
-U 1 1 5AC4EED7
-P 5050 1750
-F 0 "U2" H 4650 2400 60  0000 C CNN
-F 1 "MCP2515-I/P" H 4900 2300 60  0000 C CNN
-F 2 "IC_Sockets:IC_socket_18pins" H 6300 1250 60  0001 C CNN
-F 3 "" H 6300 1250 60  0001 C CNN
-	1    5050 1750
-	1    0    0    -1
-$EndComp
-$Comp
 L D D1
 U 1 1 5ACCAAED
@@
 F 0 "D1" H 7800 4700 50  0000 C CNN
 F 1 "1A" H 7800 4500 50  0000 C CNN
-F 2 "diode:diode" H 7800 4600 50  0001 C CNN
+F 2 "can-bus:Diode" H 7800 4600 50  0001 C CNN
 F 3 "" H 7800 4600 50  0001 C CNN
 	1    7800 4600
@@
 F 0 "F1" V 8000 4850 50  0000 C CNN
 F 1 "250mA" V 8200 4850 50  0000 C CNN
-F 2 "polyswitch:polyswitch" H 8150 4650 50  0001 L CNN
+F 2 "can-bus:Polyswitch_Tyco" H 8150 4650 50  0001 L CNN
 F 3 "" H 8100 4850 50  0001 C CNN
 	1    8100 4850
@@
 F 0 "J6" H 7300 3700 50  0000 C CNN
 F 1 "ICSP" H 7300 3000 50  0000 C CNN
-F 2 "" H 7300 3400 50  0001 C CNN
+F 2 "can-bus:PinSocket_1x6" H 7300 3400 50  0001 C CNN
 F 3 "" H 7300 3400 50  0001 C CNN
 	1    7300 3400
@@
 F 0 "J2" H 2250 3850 50  0000 C CNN
 F 1 "Pin socket" H 2250 3350 50  0000 C CNN
-F 2 "" H 2250 3650 50  0001 C CNN
+F 2 "can-bus:PinSocket_1x4" H 2250 3650 50  0001 C CNN
 F 3 "" H 2250 3650 50  0001 C CNN
 	1    2250 3650
@@
 F 0 "J3" H 2250 4650 50  0000 C CNN
 F 1 "Pin socket" H 2250 4150 50  0000 C CNN
-F 2 "" H 2250 4450 50  0001 C CNN
+F 2 "can-bus:PinSocket_1x4" H 2250 4450 50  0001 C CNN
 F 3 "" H 2250 4450 50  0001 C CNN
 	1    2250 4450
@@
 F 0 "J4" H 4400 6100 50  0000 C CNN
 F 1 "CAN0" H 4400 5800 50  0000 C CNN
-F 2 "" H 4400 6000 50  0001 C CNN
+F 2 "can-bus:PinHeader_1x2_L_Shape" H 4400 6000 50  0001 C CNN
 F 3 "" H 4400 6000 50  0001 C CNN
 	1    4400 6000
@@
 F 0 "J5" H 4400 6550 50  0000 C CNN
 F 1 "CAN1" H 4400 6250 50  0000 C CNN
-F 2 "" H 4400 6450 50  0001 C CNN
+F 2 "can-bus:PinHeader_1x2_L_Shape" H 4400 6450 50  0001 C CNN
 F 3 "" H 4400 6450 50  0001 C CNN
 	1    4400 6450
@@
 F 0 "U1" H 4300 4800 60  0000 C CNN
 F 1 "PIC16f18326-I/P" H 4600 4700 60  0000 C CNN
-F 2 "IC_Sockets:IC_socket_14pins" H 4600 4700 60  0001 C CNN
+F 2 "can-bus:IC_socket_14pins" H 4600 4700 60  0001 C CNN
 F 3 "" H 4600 4700 60  0001 C CNN
 	1    4700 4250
@@
 F 0 "U4" H 8850 4000 60  0000 C CNN
 F 1 "regulator" H 8950 3900 60  0000 C CNN
-F 2 "" H 8950 3800 60  0001 C CNN
+F 2 "can-bus:TA48M05F" H 8950 3800 60  0001 C CNN
 F 3 "" H 8950 3800 60  0001 C CNN
 	1    8950 3750
@@
 F 0 "C5" H 9460 4020 50  0000 L CNN
 F 1 "0.1u" H 9460 3870 50  0000 L CNN
-F 2 "" H 9450 3950 50  0001 C CNN
+F 2 "can-bus:Capacitor_2.54mm" H 9450 3950 50  0001 C CNN
 F 3 "" H 9450 3950 50  0001 C CNN
 	1    9450 3950
@@
 P 8450 3950
 F 0 "C4" H 8475 4050 50  0000 L CNN
-F 1 "100u" H 8475 3850 50  0000 L CNN
-F 2 "" H 8488 3800 50  0001 C CNN
+F 1 "47u" H 8475 3850 50  0000 L CNN
+F 2 "can-bus:Capacitor_2.54mm" H 8488 3800 50  0001 C CNN
 F 3 "" H 8450 3950 50  0001 C CNN
 	1    8450 3950
@@
 F 0 "J7" H 10450 3800 50  0000 C CNN
 F 1 "terminal" H 10450 3500 50  0000 C CNN
-F 2 "" H 10450 3700 50  0001 C CNN
+F 2 "can-bus:Terminal_PhoenixContact_2P" H 10450 3700 50  0001 C CNN
 F 3 "" H 10450 3700 50  0001 C CNN
 	1    10450 3700
@@
 F 0 "F2" V 9900 3700 50  0000 C CNN
 F 1 "250mA" V 10100 3700 50  0000 C CNN
-F 2 "polyswitch:polyswitch" H 10050 3500 50  0001 L CNN
+F 2 "can-bus:Polyswitch_Tyco" H 10050 3500 50  0001 L CNN
 F 3 "" H 10000 3700 50  0001 C CNN
 	1    10000 3700
@@
 F 0 "D2" H 9750 4050 50  0000 C CNN
 F 1 "1A" H 9750 3850 50  0000 C CNN
-F 2 "diode:diode" H 9750 3950 50  0001 C CNN
+F 2 "can-bus:Diode" H 9750 3950 50  0001 C CNN
 F 3 "" H 9750 3950 50  0001 C CNN
 	1    9750 3950
@@
 	6850 5400 8400 5400
 Wire Wire Line
-	1750 2150 1700 2150
-Wire Wire Line
 	1700 2150 1700 1350
 Wire Wire Line
@@
 Wire Wire Line
 	1350 1450 1350 2450
-Wire Wire Line
-	1350 2450 1750 2450
 Connection ~ 4250 2750
 Connection ~ 2850 2750
@@
 F 0 "SW1" H 4350 5600 50  0000 L CNN
 F 1 "SW" H 4300 5440 50  0000 C CNN
-F 2 "" H 4300 5700 50  0001 C CNN
+F 2 "can-bus:TactileSwitch" H 4300 5700 50  0001 C CNN
 F 3 "" H 4300 5700 50  0001 C CNN
 	1    4300 5500
@@
 F 0 "R5" V 4030 5150 50  0000 C CNN
 F 1 "1k" V 3950 5150 50  0000 C CNN
-F 2 "Resistor:Resistor_FaithfulLink_CF25" V 3880 5150 50  0001 C CNN
+F 2 "can-bus:Resistor_FaithfulLink_CF25" V 3880 5150 50  0001 C CNN
 F 3 "" H 3950 5150 50  0001 C CNN
 	1    3950 5150
@@
 F 0 "D3" H 4350 5250 50  0000 C CNN
 F 1 "LED" H 4350 5050 50  0000 C CNN
-F 2 "" H 4350 5150 50  0001 C CNN
+F 2 "can-bus:Led" H 4350 5150 50  0001 C CNN
 F 3 "" H 4350 5150 50  0001 C CNN
 	1    4350 5150
@@
 F 0 "JP2" H 4800 5230 50  0000 C CNN
 F 1 "Jumper" H 4810 5090 50  0000 C CNN
-F 2 "Connector_PinHeader_2.54mm:Jumper_1x2" H 4800 5150 50  0001 C CNN
+F 2 "can-bus:Jumper_1x2" H 4800 5150 50  0001 C CNN
 F 3 "" H 4800 5150 50  0001 C CNN
 	1    4800 5150
@@
 	7550 5200 8400 5200
 Connection ~ 7550 5200
+$Comp
+L MCP2515-I/P U3
+U 1 1 5ACEEDEE
+P 5050 1750
+F 0 "U3" H 4650 2400 60  0000 C CNN
+F 1 "MCP2515-I/P" H 4900 2300 60  0000 C CNN
+F 2 "can-bus:IC_socket_18pins" H 6300 1250 60  0001 C CNN
+F 3 "" H 6300 1250 60  0001 C CNN
+	1    5050 1750
+	1    0    0    -1
+$EndComp
+$Comp
+L MCP2561-E/P U2
+U 1 1 5ACEEE4B
+P 2400 2550
+F 0 "U2" H 2000 3200 60  0000 C CNN
+F 1 "MCP2561-E/P" H 2250 3100 60  0000 C CNN
+F 2 "can-bus:IC_Socket_8pins" H 2400 2550 60  0001 C CNN
+F 3 "" H 2400 2550 60  0001 C CNN
+	1    2400 2550
+	1    0    0    -1
+$EndComp
+Wire Wire Line
+	1350 2450 1750 2450
+Wire Wire Line
+	1700 2150 1750 2150
 $EndSCHEMATC
