File: KiCAD/circuit/adapter.sch (KiCad schematic (older format))
At the start: 29 parts, among them J1 Pin header, J2 Pin socket, J3 Pin socket, J4 CAN0, J5 CAN1, J6 ICSP, J7 terminal, SW1 SW, U1 PIC16f18326-I/P, U2 MCP2561-E/P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

Commit message: update
Parts:
- removed D2: 1A, can-bus:Diode, symbol D
- U4: value regulator -> TA48M05F
Other:
- moved on the sheet: F2, J7
Changed lines of the file:
@@
 $EndComp
 $Comp
-L +5V #PWR12
+L +5V #PWR01
 U 1 1 5AC4A3F8
 P 8100 3300
-F 0 "#PWR12" H 8100 3150 50  0001 C CNN
+F 0 "#PWR01" H 8100 3150 50  0001 C CNN
 F 1 "+5V" H 8100 3440 50  0000 C CNN
 F 2 "" H 8100 3300 50  0001 C CNN
@@
 $EndComp
 $Comp
-L GND #PWR11
+L GND #PWR02
 U 1 1 5AC4A426
 P 7550 6000
-F 0 "#PWR11" H 7550 5750 50  0001 C CNN
+F 0 "#PWR02" H 7550 5750 50  0001 C CNN
 F 1 "GND" H 7550 5850 50  0000 C CNN
 F 2 "" H 7550 6000 50  0001 C CNN
@@
 $EndComp
 $Comp
-L PWR_FLAG #FLG2
+L PWR_FLAG #FLG03
 U 1 1 5AC4A64D
 P 8500 3400
-F 0 "#FLG2" H 8500 3475 50  0001 C CNN
+F 0 "#FLG03" H 8500 3475 50  0001 C CNN
 F 1 "PWR_FLAG" H 8500 3550 50  0000 C CNN
 F 2 "" H 8500 3400 50  0001 C CNN
@@
 $EndComp
 $Comp
-L PWR_FLAG #FLG1
+L PWR_FLAG #FLG04
 U 1 1 5AC4A67B
 P 7950 5850
-F 0 "#FLG1" H 7950 5925 50  0001 C CNN
+F 0 "#FLG04" H 7950 5925 50  0001 C CNN
 F 1 "PWR_FLAG" H 7950 6000 50  0000 C CNN
 F 2 "" H 7950 5850 50  0001 C CNN
@@
 $EndComp
 $Comp
-L +5V #PWR5
+L +5V #PWR05
 U 1 1 5AC4B26C
 P 4050 3100
-F 0 "#PWR5" H 4050 2950 50  0001 C CNN
+F 0 "#PWR05" H 4050 2950 50  0001 C CNN
 F 1 "+5V" H 4050 3240 50  0000 C CNN
 F 2 "" H 4050 3100 50  0001 C CNN
@@
 $EndComp
 $Comp
-L GND #PWR9
+L GND #PWR06
 U 1 1 5AC4B2B4
 P 6150 3700
-F 0 "#PWR9" H 6150 3450 50  0001 C CNN
+F 0 "#PWR06" H 6150 3450 50  0001 C CNN
 F 1 "GND" H 6150 3550 50  0000 C CNN
 F 2 "" H 6150 3700 50  0001 C CNN
@@
 $EndComp
 $Comp
-L +5V #PWR1
+L +5V #PWR07
 U 1 1 5AC4B51B
 P 1550 2000
-F 0 "#PWR1" H 1550 1850 50  0001 C CNN
+F 0 "#PWR07" H 1550 1850 50  0001 C CNN
 F 1 "+5V" H 1550 2140 50  0000 C CNN
 F 2 "" H 1550 2000 50  0001 C CNN
@@
 $EndComp
 $Comp
-L GND #PWR2
+L GND #PWR08
 U 1 1 5AC4B5F0
 P 1550 3050
-F 0 "#PWR2" H 1550 2800 50  0001 C CNN
+F 0 "#PWR08" H 1550 2800 50  0001 C CNN
 F 1 "GND" H 1550 2900 50  0000 C CNN
 F 2 "" H 1550 3050 50  0001 C CNN
@@
 $EndComp
 $Comp
-L +5V #PWR8
+L +5V #PWR09
 U 1 1 5AC4B724
 P 6000 1050
-F 0 "#PWR8" H 6000 900 50  0001 C CNN
+F 0 "#PWR09" H 6000 900 50  0001 C CNN
 F 1 "+5V" H 6000 1190 50  0000 C CNN
 F 2 "" H 6000 1050 50  0001 C CNN
@@
 $EndComp
 $Comp
-L GND #PWR10
+L GND #PWR010
 U 1 1 5AC4B7D1
 P 7000 1750
-F 0 "#PWR10" H 7000 1500 50  0001 C CNN
+F 0 "#PWR010" H 7000 1500 50  0001 C CNN
 F 1 "GND" H 7000 1600 50  0000 C CNN
 F 2 "" H 7000 1750 50  0001 C CNN
@@
 $EndComp
 $Comp
-L +5V #PWR3
+L +5V #PWR011
 U 1 1 5ACD2D21
 P 2750 3200
-F 0 "#PWR3" H 2750 3050 50  0001 C CNN
+F 0 "#PWR011" H 2750 3050 50  0001 C CNN
 F 1 "+5V" H 2750 3340 50  0000 C CNN
 F 2 "" H 2750 3200 50  0001 C CNN
@@
 $EndComp
 $Comp
-L GND #PWR4
+L GND #PWR012
 U 1 1 5ACD2D5B
 P 2750 3850
-F 0 "#PWR4" H 2750 3600 50  0001 C CNN
+F 0 "#PWR012" H 2750 3600 50  0001 C CNN
 F 1 "GND" H 2750 3700 50  0000 C CNN
 F 2 "" H 2750 3850 50  0001 C CNN
@@
 P 8950 3750
 F 0 "U4" H 8850 4000 60  0000 C CNN
-F 1 "regulator" H 8950 3900 60  0000 C CNN
+F 1 "TA48M05F" H 8950 3900 60  0000 C CNN
 F 2 "can-bus:TA48M05F" H 8950 3800 60  0001 C CNN
 F 3 "" H 8950 3800 60  0001 C CNN
@@
 L Screw_Terminal_01x02 J7
 U 1 1 5ACEDCC0
-P 10450 3700
-F 0 "J7" H 10450 3800 50  0000 C CNN
-F 1 "terminal" H 10450 3500 50  0000 C CNN
-F 2 "can-bus:Terminal_PhoenixContact_2P" H 10450 3700 50  0001 C CNN
-F 3 "" H 10450 3700 50  0001 C CNN
-	1    10450 3700
-	1    0    0    -1
-$EndComp
-$Comp
-L GND #PWR13
+P 10350 3700
+F 0 "J7" H 10350 3800 50  0000 C CNN
+F 1 "terminal" H 10350 3500 50  0000 C CNN
+F 2 "can-bus:Terminal_PhoenixContact_2P" H 10350 3700 50  0001 C CNN
+F 3 "" H 10350 3700 50  0001 C CNN
+	1    10350 3700
+	1    0    0    -1
+$EndComp
+$Comp
+L GND #PWR013
 U 1 1 5ACED80E
 P 10150 4550
-F 0 "#PWR13" H 10150 4300 50  0001 C CNN
+F 0 "#PWR013" H 10150 4300 50  0001 C CNN
 F 1 "GND" H 10150 4400 50  0000 C CNN
 F 2 "" H 10150 4550 50  0001 C CNN
@@
 L Polyfuse F2
 U 1 1 5ACEE675
-P 10000 3700
-F 0 "F2" V 9900 3700 50  0000 C CNN
-F 1 "250mA" V 10100 3700 50  0000 C CNN
-F 2 "can-bus:Polyswitch_Tyco" H 10050 3500 50  0001 L CNN
-F 3 "" H 10000 3700 50  0001 C CNN
-	1    10000 3700
+P 9850 3700
+F 0 "F2" V 9750 3700 50  0000 C CNN
+F 1 "250mA" V 9950 3700 50  0000 C CNN
+F 2 "can-bus:Polyswitch_Tyco" H 9900 3500 50  0001 L CNN
+F 3 "" H 9850 3700 50  0001 C CNN
+	1    9850 3700
 	0    1    1    0
 $EndComp
-$Comp
-L D D2
-U 1 1 5ACEE9DD
-P 9750 3950
-F 0 "D2" H 9750 4050 50  0000 C CNN
-F 1 "1A" H 9750 3850 50  0000 C CNN
-F 2 "can-bus:Diode" H 9750 3950 50  0001 C CNN
-F 3 "" H 9750 3950 50  0001 C CNN
-	1    9750 3950
-	0    -1   1    0
-$EndComp
 Wire Wire Line
 	1250 2250 1250 2750
@@
 	4050 3100 4050 3950
 Wire Wire Line
-	6450 4550 6000 4550
-Wire Wire Line
-	6550 1650 6550 4450
-Wire Wire Line
-	6350 1850 5700 1850
+	6500 4550 6000 4550
+Wire Wire Line
+	6600 1650 6600 4450
+Wire Wire Line
+	6400 1850 5700 1850
 Wire Wire Line
 	6300 1550 5700 1550
@@
 	5700 1450 6500 1450
 Wire Wire Line
-	6550 4450 6000 4450
-Wire Wire Line
-	6550 1650 5700 1650
-Wire Wire Line
-	5700 1750 6450 1750
-Wire Wire Line
-	6450 1750 6450 4550
-Wire Wire Line
-	6350 1850 6350 4350
-Wire Wire Line
-	6350 4350 6000 4350
+	6600 4450 6000 4450
+Wire Wire Line
+	6600 1650 5700 1650
+Wire Wire Line
+	5700 1750 6500 1750
+Wire Wire Line
+	6500 1750 6500 4550
+Wire Wire Line
+	6400 1850 6400 4350
+Wire Wire Line
+	6400 4350 6000 4350
 Wire Wire Line
 	6300 1550 6300 4250
@@
 	8100 3700 8500 3700
 Wire Wire Line
-	9400 3700 9850 3700
-Wire Wire Line
 	8450 4100 8450 4250
 Wire Wire Line
@@
 	8450 3800 8450 3700
 Connection ~ 8450 3700
-Wire Wire Line
-	10250 3800 10150 3800
 Wire Wire Line
 	10150 3800 10150 4550
@@
 Connection ~ 8100 3700
 Wire Wire Line
-	10150 3700 10250 3700
-Wire Wire Line
-	9750 3800 9750 3700
-Connection ~ 9750 3700
-Wire Wire Line
-	9750 4100 9750 4250
-Connection ~ 9750 4250
+	10000 3700 10150 3700
 Wire Wire Line
 	3500 5500 4100 5500
@@
 $EndComp
 $Comp
-L GND #PWR7
+L GND #PWR014
 U 1 1 5ACEDE89
 P 5250 5650
-F 0 "#PWR7" H 5250 5400 50  0001 C CNN
+F 0 "#PWR014" H 5250 5400 50  0001 C CNN
 F 1 "GND" H 5250 5500 50  0000 C CNN
 F 2 "" H 5250 5650 50  0001 C CNN
@@
 	5250 5500 5250 5650
 $Comp
-L +5V #PWR6
+L +5V #PWR015
 U 1 1 5ACEE4D3
 P 5250 4950
-F 0 "#PWR6" H 5250 4800 50  0001 C CNN
+F 0 "#PWR015" H 5250 4800 50  0001 C CNN
 F 1 "+5V" H 5250 5090 50  0000 C CNN
 F 2 "" H 5250 4950 50  0001 C CNN
@@
 Wire Wire Line
 	1700 2150 1750 2150
+Wire Wire Line
+	9400 3700 9700 3700
 $EndSCHEMATC
