File: KiCAD/circuit/doppler/doppler.sch (KiCad schematic (older format))
At the start: 7 parts, among them J1 Conn_01x04_Male, J2 Conn_01x04_Male, U1 Doppler_sensor

Commit message: update
Parts:
- D1, D2: footprint (none) -> can-bus:Led
- J1, J2: footprint (none) -> can-bus:PinHeader_1x4
- R1, R2: footprint (none) -> can-bus:Resistor_FaithfulLink_CF25
- U1: footprint (none) -> can-bus:Doppler_sensor_NJR4265_J1
Changed lines of the file:
@@
 F 0 "U1" H 4850 4600 60  0000 C CNN
 F 1 "Doppler_sensor" H 5700 4200 60  0000 C CNN
-F 2 "" V 4800 4250 60  0001 C CNN
+F 2 "can-bus:Doppler_sensor_NJR4265_J1" V 4800 4250 60  0001 C CNN
 F 3 "" V 4800 4250 60  0001 C CNN
 	1    5700 4050
@@
 $EndComp
 $Comp
-L GND #PWR4
+L GND #PWR01
 U 1 1 5AD94916
 P 7500 4400
-F 0 "#PWR4" H 7500 4150 50  0001 C CNN
+F 0 "#PWR01" H 7500 4150 50  0001 C CNN
 F 1 "GND" H 7500 4250 50  0000 C CNN
 F 2 "" H 7500 4400 50  0001 C CNN
@@
 	7500 3250 7500 4400
 $Comp
-L PWR_FLAG #FLG2
+L PWR_FLAG #FLG02
 U 1 1 5AD9494A
 P 7850 4150
-F 0 "#FLG2" H 7850 4225 50  0001 C CNN
+F 0 "#FLG02" H 7850 4225 50  0001 C CNN
 F 1 "PWR_FLAG" H 7850 4300 50  0000 C CNN
 F 2 "" H 7850 4150 50  0001 C CNN
@@
 F 0 "J1" H 5550 2650 50  0000 C CNN
 F 1 "Conn_01x04_Male" H 5550 2150 50  0000 C CNN
-F 2 "" H 5550 2450 50  0001 C CNN
+F 2 "can-bus:PinHeader_1x4" H 5550 2450 50  0001 C CNN
 F 3 "" H 5550 2450 50  0001 C CNN
 	1    5550 2450
@@
 F 0 "J2" H 5700 5700 50  0000 C CNN
 F 1 "Conn_01x04_Male" H 5700 5200 50  0000 C CNN
-F 2 "" H 5700 5500 50  0001 C CNN
+F 2 "can-bus:PinHeader_1x4" H 5700 5500 50  0001 C CNN
 F 3 "" H 5700 5500 50  0001 C CNN
 	1    5700 5500
@@
 	5450 3250 5450 2650
 $Comp
-L +5V #PWR1
+L +5V #PWR03
 U 1 1 5AD94ED8
 P 4000 2900
-F 0 "#PWR1" H 4000 2750 50  0001 C CNN
+F 0 "#PWR03" H 4000 2750 50  0001 C CNN
 F 1 "+5V" H 4000 3040 50  0000 C CNN
 F 2 "" H 4000 2900 50  0001 C CNN
@@
 Connection ~ 4000 3250
 $Comp
-L PWR_FLAG #FLG1
+L PWR_FLAG #FLG04
 U 1 1 5AD94F0E
 P 3600 2900
-F 0 "#FLG1" H 3600 2975 50  0001 C CNN
+F 0 "#FLG04" H 3600 2975 50  0001 C CNN
 F 1 "PWR_FLAG" H 3600 3050 50  0000 C CNN
 F 2 "" H 3600 2900 50  0001 C CNN
@@
 F 0 "D1" H 4400 5500 50  0000 C CNN
 F 1 "LED" H 4400 5300 50  0000 C CNN
-F 2 "" H 4400 5400 50  0001 C CNN
+F 2 "can-bus:Led" H 4400 5400 50  0001 C CNN
 F 3 "" H 4400 5400 50  0001 C CNN
 	1    4400 5400
@@
 F 0 "D2" H 4700 5500 50  0000 C CNN
 F 1 "LED" H 4700 5300 50  0000 C CNN
-F 2 "" H 4700 5400 50  0001 C CNN
+F 2 "can-bus:Led" H 4700 5400 50  0001 C CNN
 F 3 "" H 4700 5400 50  0001 C CNN
 	1    4700 5400
@@
 F 0 "R1" V 4480 5900 50  0000 C CNN
 F 1 "1k" V 4400 5900 50  0000 C CNN
-F 2 "" V 4330 5900 50  0001 C CNN
+F 2 "can-bus:Resistor_FaithfulLink_CF25" V 4330 5900 50  0001 C CNN
 F 3 "" H 4400 5900 50  0001 C CNN
 	1    4400 5900
@@
 F 0 "R2" V 4780 5900 50  0000 C CNN
 F 1 "1k" V 4700 5900 50  0000 C CNN
-F 2 "" V 4630 5900 50  0001 C CNN
+F 2 "can-bus:Resistor_FaithfulLink_CF25" V 4630 5900 50  0001 C CNN
 F 3 "" H 4700 5900 50  0001 C CNN
 	1    4700 5900
@@
 $EndComp
 $Comp
-L GND #PWR2
+L GND #PWR05
 U 1 1 5AD953A8
 P 4400 6300
-F 0 "#PWR2" H 4400 6050 50  0001 C CNN
+F 0 "#PWR05" H 4400 6050 50  0001 C CNN
 F 1 "GND" H 4400 6150 50  0000 C CNN
 F 2 "" H 4400 6300 50  0001 C CNN
@@
 $EndComp
 $Comp
-L GND #PWR3
+L GND #PWR06
 U 1 1 5AD953CA
 P 4700 6300
-F 0 "#PWR3" H 4700 6050 50  0001 C CNN
+F 0 "#PWR06" H 4700 6050 50  0001 C CNN
 F 1 "GND" H 4700 6150 50  0000 C CNN
 F 2 "" H 4700 6300 50  0001 C CNN
